File: Hardware/Production/USB-C_Host_Shield-Panel.brd (EAGLE design)
At the start: 120.9 x 301.8 mm, 878 parts, among them J1 USB-C, J10 USB-C, J11 GPIN, J12 GPOUT, J13 USB-C, J14 GPIN, J15 GPOUT, J16 USB-C, J17 GPIN, J18 GPOUT, J19 USB-C, J2 GPIN, J20 GPIN, J21 GPOUT, J22 USB-C, J23 GPIN, J24 GPOUT, J3 GPOUT, J4 USB-C, J5 GPIN, J6 GPOUT, J7 USB-C, J8 GPIN, J9 GPOUT, U1 ARDUINO_UNO_R3_SHIELDNOLABELS, U10 ARDUINO_UNO_R3_SHIELDNOLABELS, U11 LM1117, U12 74HC4050, U13 3.3V/150mA, U14 MAX3421, U15 ARDUINO_UNO_R3_SHIELDNOLABELS, U16 LM1117, U17 74HC4050, U18 3.3V/150mA, U19 MAX3421, U2 LM1117, U20 ARDUINO_UNO_R3_SHIELDNOLABELS, U21 LM1117, U22 74HC4050, U23 3.3V/150mA, U24 MAX3421, U25 ARDUINO_UNO_R3_SHIELDNOLABELS, U26 LM1117, U27 74HC4050, U28 3.3V/150mA, U29 MAX3421, U3 74HC4050, U30 ARDUINO_UNO_R3_SHIELDNOLABELS, U31 LM1117, U32 74HC4050, U33 3.3V/150mA, U34 MAX3421, U35 ARDUINO_UNO_R3_SHIELDNOLABELS, U36 LM1117, U37 74HC4050, U38 3.3V/150mA, U39 MAX3421, U4 LM1117, U40 ARDUINO_UNO_R3_SHIELDNOLABELS, U5 MAX3421, U6 3.3V/150mA, U7 74HC4050, U8 3.3V/150mA, U9 MAX3421, Y1 12.0mhZ, Y2 12.0mhZ, Y3 12.0mhZ, Y4 12.0mhZ, Y5 12.0mhZ, Y6 12.0mhZ, Y7 12.0mhZ, Y8 12.0mhZ

Commit message: Added panel files and adjusted schematic notation
Ran panelization script and added those files to the repo. Adjusted the Vin input value on the schematic for people to better understand the input range.
Parts:
- removed D10, D12, D14, D16: 1A/15V/220mV, SparkFun-DiscreteSemi:DO-214BA
- removed D11, D13, D15, D9: RED, SparkFun-LED:LED-0603
- added U$505, U$599, U$693: (no value), output:RX13
- added U$506, U$600, U$694: (no value), output:TX1131211211109876543245
- added U$507, U$515, U$601, U$609, U$695, U$703: (no value), output:21131211211109876543246
- added U$508, U$516, U$602, U$610, U$696, U$704: (no value), output:321131211211109876543247
- added U$509, U$517, U$603, U$611, U$697, U$705: (no value), output:4321131211211109876543248
- added U$510, U$518, U$604, U$612, U$698, U$706: (no value), output:54321131211211109876543249
- added U$511, U$605, U$699: (no value), output:654321131211211109876543250
- added U$512, U$606, U$700: (no value), output:7654321131211211109876543251
- added U$513, U$607, U$701: (no value), output:17654321131211211109876543252
- added U$514, U$608, U$702: (no value), output:017654321131211211109876543253
- added U$519, U$613, U$707: (no value), output:817654321131211211109876543254
- added U$520, U$614, U$708: (no value), output:9817654321131211211109876543255
- added U$521, U$615, U$709: (no value), output:109817654321131211211109876543256
- added U$522, U$616, U$710: (no value), output:11109817654321131211211109876543257
- added U$523, U$617, U$711: (no value), output:1211109817654321131211211109876543258
- added U$524, U$618, U$712: (no value), output:131211109817654321131211211109876543259
- added U$525, U$526, U$619, U$620, U$713, U$714: (no value), output:GND131211109817654321131211211109876543260
- added U$527, U$621, U$715: (no value), output:SDA131211109817654321131211211109876543261
- added U$528, U$622, U$716: (no value), output:SCL131211109817654321131211211109876543262
- added U$529, U$623, U$717: (no value), output:IOREF131211109817654321131211211109876543264
- added U$530, U$624, U$718: (no value), output:RST131211109817654321131211211109876543265
- added U$531, U$625, U$719: (no value), output:#3#3V4
- added U$532, U$626, U$720: (no value), output:#5V4
- added U$533, U$627, U$721: (no value), output:VIN6
- added U$534, U$628, U$722: (no value), output:#_5#6
- added U$535, U$629, U$723: (no value), output:#_4#6
- added U$536, U$630, U$724: (no value), output:#_3#6
- added U$537, U$631, U$725: (no value), output:#_2#6
- added U$538, U$632, U$726: (no value), output:#_1#6
- added U$539, U$633, U$727: (no value), output:#_0#6
- added U$540, U$634, U$728: (no value), output:#_VIN#6
- added U$541, U$542, U$635, U$636, U$729, U$730: (no value), output:#_GND#7
- added U$543, U$637, U$731: (no value), output:#_#5V#8
- added U$544, U$638, U$732: (no value), output:#_#3#3V#8
- added U$545, U$639, U$733: (no value), output:#_RST#8
- added U$546, U$640, U$734: (no value), output:#_IOREF#9
- added U$547, U$641, U$735: (no value), output:#RX_#10
- added U$548, U$642, U$736: (no value), output:#TX_#11
- added U$549, U$643, U$737: (no value), output:#2_#12
- added U$550, U$644, U$738: (no value), output:#3_#12
- added U$551, U$645, U$739: (no value), output:#4_#12
- added U$552, U$646, U$740: (no value), output:#5_#12
- added U$553, U$647, U$741: (no value), output:#6_#12
- added U$554, U$648, U$742: (no value), output:#7#RESET_#12
- added U$555, U$649, U$743: (no value), output:#8#GPX_#12
- added U$556, U$650, U$744: (no value), output:#9#INT_#12
- added U$557, U$651, U$745: (no value), output:#10#CS_#12
- added U$558, U$652, U$746: (no value), output:#11#PICO_#12
- added U$559, U$653, U$747: (no value), output:#12#POCI_#12
- added U$560, U$654, U$748: (no value), output:#13#SCK_#13
- added U$561, U$655, U$749: (no value), output:#SDA#18
- added U$562, U$656, U$750: (no value), output:#SCL#19
- added U$563, U$657, U$751: (no value), output:#AREF#20
- added U$564, U$658, U$752: (no value), output:#GND#21
- added U$565, U$659: (no value), output:POWER23
- added U$566, U$660: (no value), SparkFun-Aesthetics:SFE_LOGO_FLAME_.2
- added U$567, U$661: (no value), output:RESET25
- added U$568, U$662: (no value), output:ON26
- added U$569, U$663: (no value), output:OFF27
- added U$570, U$664: (no value), output:ANALOG_IN28
- added U$571, U$665: (no value), output:USB#C_HOST_SHIELD32
- added U$572, U$666: (no value), output:SHLD#33
- added U$573, U$667: (no value), output:MAIN40
- added U$574, U$668: (no value), output:POWER38
- added U$575, U$669: (no value), output:GPIN42
- added U$576, U$670: (no value), output:GPOUT44
- added U$577, U$589, U$671, U$683: (no value), output:045
- added U$578, U$590, U$672, U$684: (no value), output:146
- added U$579, U$591, U$673, U$685: (no value), output:2147
- added U$580, U$592, U$674, U$686: (no value), output:32148
- added U$581, U$582, U$675, U$676: (no value), output:4332150
- added U$583, U$584, U$677, U$678: (no value), output:54332151
- added U$585, U$586, U$679, U$680: (no value), output:654332152
- added U$587, U$588, U$681, U$682: (no value), output:7654332153
- added U$593, U$687: (no value), output:5V6
- added U$594, U$688: (no value), output:VIN7
- added U$595, U$689: (no value), output:POWER11
- added U$596, U$690: (no value), output:SELECT12
- added U$597, U$691: (no value), output:GND131211211109876543229
- added U$598, U$692: (no value), output:AREF131211211109876543230
- C11: value 2.2uF -> 10uF
- C13, C24, C35, C46, C57, C68, C79: value 2.2uF -> 10uF; device SparkFun-Capacitors:0603 -> SparkFun-Capacitors:EIA3216
- C15, C26, C37, C48, C59, C70, C81: device SparkFun-Capacitors:EIA3216 -> SparkFun-Capacitors:0603
- C16, C27, C38, C49, C60, C71, C82: value 10uF -> 18pF
- C17, C28, C39, C50, C61, C72, C83: value 18pF -> 0.1uF
- C22, C33, C44, C55, C66, C77, C88: value 0.1uF -> 10uF
- D2, D4, D6, D8: value 1A/15V/220mV -> RED; device SparkFun-DiscreteSemi:DO-214BA -> SparkFun-LED:LED-0603
- F1, F2, F3, F4, F5, F6, F7, F8: value 6V/0.5A -> 6V/0.75A
- U$100: device output:21131211211109876543246 -> output:ANALOG_IN28
- U$101: device output:321131211211109876543247 -> output:USB#C_HOST_SHIELD32
- U$102: device output:4321131211211109876543248 -> output:SHLD#33
- U$103: device output:54321131211211109876543249 -> output:MAIN40
- U$104: device output:654321131211211109876543250 -> output:POWER38
- U$105: device output:7654321131211211109876543251 -> output:GPIN42
- U$106: device output:17654321131211211109876543252 -> output:GPOUT44
- U$107: device output:017654321131211211109876543253 -> output:045
- U$108: device output:21131211211109876543246 -> output:146
- U$109: device output:321131211211109876543247 -> output:2147
- U$110: device output:4321131211211109876543248 -> output:32148
- U$111, U$300: device output:54321131211211109876543249 -> output:4332150
- U$112: device output:817654321131211211109876543254 -> output:4332150
- U$113, U$302: device output:9817654321131211211109876543255 -> output:54332151
- U$114: device output:109817654321131211211109876543256 -> output:54332151
- U$115, U$304: device output:11109817654321131211211109876543257 -> output:654332152
- U$116: device output:1211109817654321131211211109876543258 -> output:654332152
- U$117, U$306: device output:131211109817654321131211211109876543259 -> output:7654332153
- U$118: device output:GND131211109817654321131211211109876543260 -> output:7654332153
- U$119, U$307: device output:GND131211109817654321131211211109876543260 -> output:045
- U$120: device output:SDA131211109817654321131211211109876543261 -> output:146
- U$121: device output:SCL131211109817654321131211211109876543262 -> output:2147
- U$122: device output:IOREF131211109817654321131211211109876543264 -> output:32148
- U$123: device output:RST131211109817654321131211211109876543265 -> output:5V6
- U$124: device output:#3#3V4 -> output:VIN7
- U$125: device output:#5V4 -> output:POWER11
- U$126: device output:VIN6 -> output:SELECT12
- U$127: device output:POWER23 -> output:GND131211211109876543229
- U$128: device SparkFun-Aesthetics:SFE_LOGO_FLAME_.2 -> output:AREF131211211109876543230
- U$129: device output:RESET25 -> output:RX13
- U$130: device output:ON26 -> output:TX1131211211109876543245
- U$131: device output:OFF27 -> output:21131211211109876543246
- U$132: device output:ANALOG_IN28 -> output:321131211211109876543247
- U$133: device output:USB#C_HOST_SHIELD32 -> output:4321131211211109876543248
- U$134: device output:SHLD#33 -> output:54321131211211109876543249
- U$135: device output:MAIN40 -> output:654321131211211109876543250
- U$136: device output:POWER38 -> output:7654321131211211109876543251
- U$137: device output:GPIN42 -> output:17654321131211211109876543252
- U$138: device output:GPOUT44 -> output:017654321131211211109876543253
- U$139: device output:045 -> output:21131211211109876543246
- U$140: device output:146 -> output:321131211211109876543247
- U$141: device output:2147 -> output:4321131211211109876543248
- U$142: device output:32148 -> output:54321131211211109876543249
- U$143: device output:4332150 -> output:817654321131211211109876543254
- U$144, U$332: device output:4332150 -> output:9817654321131211211109876543255
- U$145: device output:54332151 -> output:109817654321131211211109876543256
- U$146, U$334: device output:54332151 -> output:11109817654321131211211109876543257
- U$147: device output:654332152 -> output:1211109817654321131211211109876543258
- U$148, U$336: device output:654332152 -> output:131211109817654321131211211109876543259
- U$149, U$150, U$338: device output:7654332153 -> output:GND131211109817654321131211211109876543260
- U$151: device output:045 -> output:SDA131211109817654321131211211109876543261
- U$152: device output:146 -> output:SCL131211109817654321131211211109876543262
- U$153: device output:2147 -> output:IOREF131211109817654321131211211109876543264
- U$154: device output:32148 -> output:RST131211109817654321131211211109876543265
- U$155: device output:5V6 -> output:#3#3V4
- U$156: device output:VIN7 -> output:#5V4
- U$157: device output:POWER11 -> output:VIN6
- U$158: device output:SELECT12 -> output:#_5#6
- U$159: device output:GND131211211109876543229 -> output:#_4#6
- U$160: device output:AREF131211211109876543230 -> output:#_3#6
- U$161: device output:RX13 -> output:#_2#6
- U$162: device output:TX1131211211109876543245 -> output:#_1#6
- U$163: device output:21131211211109876543246 -> output:#_0#6
- U$164: device output:321131211211109876543247 -> output:#_VIN#6
- U$165, U$354: device output:4321131211211109876543248 -> output:#_GND#7
- U$166: device output:54321131211211109876543249 -> output:#_GND#7
- U$167: device output:654321131211211109876543250 -> output:#_#5V#8
- U$168: device output:7654321131211211109876543251 -> output:#_#3#3V#8
- U$169: device output:17654321131211211109876543252 -> output:#_RST#8
- U$170: device output:017654321131211211109876543253 -> output:#_IOREF#9
- U$171: device output:21131211211109876543246 -> output:#RX_#10
- U$172: device output:321131211211109876543247 -> output:#TX_#11
- U$173: device output:4321131211211109876543248 -> output:#2_#12
- U$174: device output:54321131211211109876543249 -> output:#3_#12
- U$175: device output:817654321131211211109876543254 -> output:#4_#12
- U$176: device output:9817654321131211211109876543255 -> output:#5_#12
- U$177: device output:109817654321131211211109876543256 -> output:#6_#12
- U$178: device output:11109817654321131211211109876543257 -> output:#7#RESET_#12
- U$179: device output:1211109817654321131211211109876543258 -> output:#8#GPX_#12
- U$180: device output:131211109817654321131211211109876543259 -> output:#9#INT_#12
- U$181: device output:GND131211109817654321131211211109876543260 -> output:#10#CS_#12
- U$182, U$370: device output:GND131211109817654321131211211109876543260 -> output:#11#PICO_#12
- U$183: device output:SDA131211109817654321131211211109876543261 -> output:#12#POCI_#12
- U$184: device output:SCL131211109817654321131211211109876543262 -> output:#13#SCK_#13
- U$185: device output:IOREF131211109817654321131211211109876543264 -> output:#SDA#18
- U$186: device output:RST131211109817654321131211211109876543265 -> output:#SCL#19
- U$187: device output:#3#3V4 -> output:#AREF#20
- U$188: device output:#5V4 -> output:#GND#21
- U$189: device output:VIN6 -> output:POWER23
- U$190: device output:POWER23 -> SparkFun-Aesthetics:SFE_LOGO_FLAME_.2
- U$191: device SparkFun-Aesthetics:SFE_LOGO_FLAME_.2 -> output:RESET25
- U$192: device output:RESET25 -> output:ON26
- U$193: device output:ON26 -> output:OFF27
- U$194: device output:OFF27 -> output:ANALOG_IN28
- U$195: device output:ANALOG_IN28 -> output:USB#C_HOST_SHIELD32
- U$196: device output:USB#C_HOST_SHIELD32 -> output:SHLD#33
- U$197: device output:SHLD#33 -> output:MAIN40
- U$198: device output:MAIN40 -> output:POWER38
- U$199: device output:POWER38 -> output:GPIN42
- U$200: device output:GPIN42 -> output:GPOUT44
- U$201: device output:GPOUT44 -> output:045
- U$202, U$214: device output:045 -> output:146
- U$203, U$215: device output:146 -> output:2147
- U$204, U$216: device output:2147 -> output:32148
- U$205, U$394: device output:32148 -> output:4332150
- U$207, U$395, U$396: device output:4332150 -> output:54332151
- U$209, U$397, U$398: device output:54332151 -> output:654332152
- U$211, U$399, U$400: device output:654332152 -> output:7654332153
- U$213, U$401: device output:7654332153 -> output:045
- U$217: device output:32148 -> output:5V6
- U$218: device output:5V6 -> output:VIN7
- U$219: device output:VIN7 -> output:POWER11
- U$220: device output:POWER11 -> output:SELECT12
- U$221: device output:SELECT12 -> output:GND131211211109876543229
- U$222: device output:GND131211211109876543229 -> output:AREF131211211109876543230
- U$223: device output:AREF131211211109876543230 -> output:RX13
- U$224: device output:RX13 -> output:TX1131211211109876543245
- U$225: device output:TX1131211211109876543245 -> output:21131211211109876543246
- U$226, U$234: device output:21131211211109876543246 -> output:321131211211109876543247
- U$227, U$235: device output:321131211211109876543247 -> output:4321131211211109876543248
- U$228, U$236: device output:4321131211211109876543248 -> output:54321131211211109876543249
- U$229: device output:54321131211211109876543249 -> output:654321131211211109876543250
- U$230: device output:654321131211211109876543250 -> output:7654321131211211109876543251
- U$231: device output:7654321131211211109876543251 -> output:17654321131211211109876543252
- U$232: device output:17654321131211211109876543252 -> output:017654321131211211109876543253
- U$233: device output:017654321131211211109876543253 -> output:21131211211109876543246
- U$237: device output:54321131211211109876543249 -> output:817654321131211211109876543254
- U$238: device output:817654321131211211109876543254 -> output:9817654321131211211109876543255
- U$239: device output:9817654321131211211109876543255 -> output:109817654321131211211109876543256
- U$240: device output:109817654321131211211109876543256 -> output:11109817654321131211211109876543257
- U$241: device output:11109817654321131211211109876543257 -> output:1211109817654321131211211109876543258
- U$242: device output:1211109817654321131211211109876543258 -> output:131211109817654321131211211109876543259
- U$243, U$432: device output:131211109817654321131211211109876543259 -> output:GND131211109817654321131211211109876543260
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- renumbered JP1 to SHLD, JP2 to SHLD1, JP3 to SHLD2, JP4 to SHLD3, JP5 to SHLD4, JP6 to SHLD5, JP7 to SHLD6, JP8 to SHLD7
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Connections:
- removed net N$10: C13.1, R15.2, R16.1, U4.1
- removed net N$203 (its old number): C15.+, C20.1, R16.2, S6.1, U4.2, U4.4
- removed net N$207: D5.A, R21.1
- removed net N$208: C24.1, R25.2, R26.1, U11.1
- removed net N$306 (its old number): C26.+, C31.1, R26.2, S9.1, U11.2, U11.4
- removed net N$310: D7.A, R31.1
- removed net N$311: C35.1, R35.2, R36.1, U16.1
- removed net N$411: D8.C, F4.2
- removed net N$413: D9.A, R41.1
- removed net N$414: C46.1, R45.2, R46.1, U21.1
- removed net N$514: D10.C, F5.2
- removed net N$516: D11.A, R51.1
- removed net N$517: C57.1, R55.2, R56.1, U26.1
- removed net N$615: C59.+, C64.1, R56.2, S18.1, U26.2, U26.4
- removed net N$617: D12.C, F6.2
- removed net N$619: D13.A, R61.1
- removed net N$620: C68.1, R65.2, R66.1, U31.1
- removed net N$718: C70.+, C75.1, R66.2, S21.1, U31.2, U31.4
- removed net N$720: D14.C, F7.2
- removed net N$722: D15.A, R71.1
- removed net N$723: C79.1, R75.2, R76.1, U36.1
- removed net N$821: C81.+, C86.1, R76.2, S24.1, U36.2, U36.4
- removed net N$823: D16.C, F8.2
- new net N$202: C14.+, C19.1, R16.2, S6.1, U4.2, U4.4
- new net N$206: C33.1, R25.2, R26.1, U11.1
- new net N$304: C25.+, C30.1, R26.2, S9.1, U11.2, U11.4
- new net N$307: D4.A, R31.1
- new net N$406: C36.+, C41.1, R36.2, S12.1, U16.2, U16.4
- new net N$410: C55.1, R45.2, R46.1, U21.1
- new net N$508: C47.+, C52.1, R46.2, S15.1, U21.2, U21.4
- new net N$511: D6.A, R51.1
- new net N$610: C58.+, C63.1, R56.2, S18.1, U26.2, U26.4
- new net N$613: D7.A, R61.1
- new net N$614: C77.1, R65.2, R66.1, U31.1
- new net N$712: C69.+, C74.1, R66.2, S21.1, U31.2, U31.4
- new net N$715: D8.A, R71.1
- new net N$716: C88.1, R75.2, R76.1, U36.1
- new net N$814: C80.+, C85.1, R76.2, S24.1, U36.2, U36.4
- net 3.3V1: now also C15.1, C17.1, C21.1; no longer C16.1, C18.1, C22.1
- net 3.3V2: now also C26.1, C28.1, C32.1; no longer C27.1, C29.1, C33.1
- net 3.3V3: now also C37.1, C39.1, C43.1; no longer C38.1, C40.1, C44.1
- net 3.3V4: now also C48.1, C50.1, C54.1; no longer C49.1, C51.1, C55.1
- net 3.3V5: now also C59.1, C61.1, C65.1; no longer C60.1, C62.1, C66.1
- net 3.3V6: now also C70.1, C72.1, C76.1; no longer C71.1, C73.1, C77.1
- net 3.3V7: now also C81.1, C83.1, C87.1; no longer C82.1, C84.1, C88.1
- net GND1: now also C13.-, C15.2, D2.C; no longer C13.2, C15.-, D3.C
- net GND2: now also C24.-, C26.2, D3.C; no longer C24.2, C26.-, D5.C
- net GND3: now also C35.-, C37.2, D4.C; no longer C35.2, C37.-, D7.C
- net GND4: now also C46.-, C48.2, D5.C; no longer C46.2, C48.-, D9.C
- net GND5: now also C57.-, C59.2, D6.C; no longer C57.2, C59.-, D11.C
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Routing:
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
Commit message: Updated Production Files for Reds order
Regenerated panelized files for ordering after small review. Adjusted some small traces for better GND connection.
Parts:
- C11, C22, C33, C44, C55, C66, C77, C88: device SparkFun-Capacitors:0603 -> SparkFun-Capacitors:0805
- S1: value Main Power -> MOMENTARY-SWITCH-SPST-SMD-5.2MM-TALL; device SparkFun-Switches:SWITCH_DPDT_SMD_AYZ0202 -> SparkFun-Switches:TACTILE_SWITCH_SMD_5.2MM
- S11, S14, S17, S20, S23, S8: value Main Power -> Power Select
- S12, S15, S18, S21, S24, S6, S9: value Power Select -> Main Power
- S4: value MOMENTARY-SWITCH-SPST-SMD-5.2MM-TALL -> Power Select; device SparkFun-Switches:TACTILE_SWITCH_SMD_5.2MM -> SparkFun-Switches:SWITCH_DPDT_SMD_AYZ0202
- U10, U15, U20, U25, U30, U35, U40: value ARDUINO_UNO_R3_SHIELDNOLABELS -> MAX3421; device SparkFun-Boards:UNO_R3_SHIELD_NOLABELS -> SparkFun-IC-Microcontroller:TQFP32
- U14, U19, U24, U29, U34, U39, U9: value MAX3421 -> ARDUINO_UNO_R3_SHIELDNOLABELS; device SparkFun-IC-Microcontroller:TQFP32 -> SparkFun-Boards:UNO_R3_SHIELD_NOLABELS
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Connections:
- removed net N$201: S4.3, U10.RES
- removed net N$204 (its old number): S5.2, S6.2
- removed net N$303: S7.3, U15.RES
- removed net N$304: C25.+, C30.1, R26.2, S9.1, U11.2, U11.4
- removed net N$405: S10.3, U20.RES
- removed net N$406: C36.+, C41.1, R36.2, S12.1, U16.2, U16.4
- removed net N$507: S13.3, U25.RES
- removed net N$508: C47.+, C52.1, R46.2, S15.1, U21.2, U21.4
- removed net N$510: S14.2, S15.2
- removed net N$609: S16.3, U30.RES
- removed net N$610: C58.+, C63.1, R56.2, S18.1, U26.2, U26.4
- removed net N$612: S17.2, S18.2
- removed net N$711: S19.3, U35.RES
- removed net N$712: C69.+, C74.1, R66.2, S21.1, U31.2, U31.4
- removed net N$714: S20.2, S21.2
- removed net N$813: S22.3, U40.RES
- removed net N$814: C80.+, C85.1, R76.2, S24.1, U36.2, U36.4
- removed net N$816: S23.2, S24.2
- new net N$203: C14.+, C19.1, R16.2, S3.3, S3.6, U4.2, U4.4
- new net N$205: S3.2, S3.5, S6.2, S6.5
- new net N$206: S6.1, S6.4
- new net N$305: S7.3, U14.RES
- new net N$308: S8.2, S8.5, S9.2, S9.5
- new net N$309: S9.1, S9.4
- new net N$409: C36.+, C41.1, R36.2, S11.3, S11.6, U16.2, U16.4
- new net N$411: S11.2, S11.5, S12.2, S12.5
- new net N$412: S12.1, S12.4
- new net N$5: S5.1, S5.4
- new net N$511: S13.3, U24.RES
- new net N$512: C47.+, C52.1, R46.2, S14.3, S14.6, U21.2, U21.4
- new net N$514: S14.2, S14.5, S15.2, S15.5
- new net N$515: S15.1, S15.4
- new net N$614: S16.3, U29.RES
- new net N$615: C58.+, C63.1, R56.2, S17.3, S17.6, U26.2, U26.4
- new net N$617: S17.2, S17.5, S18.2, S18.5
- new net N$618: S18.1, S18.4
- new net N$717: S19.3, U34.RES
- new net N$718: C69.+, C74.1, R66.2, S20.3, S20.6, U31.2, U31.4
- new net N$720: S20.2, S20.5, S21.2, S21.5
- new net N$721: S21.1, S21.4
- new net N$820: S22.3, U39.RES
- new net N$821: C80.+, C85.1, R76.2, S23.3, S23.6, U36.2, U36.4
- new net N$823: S23.2, S23.5, S24.2, S24.5
- new net N$824: S24.1, S24.4
- net 3.3V1: now also U10.2, U10.23; no longer U9.2, U9.23
- net 3.3V2: now also U15.2, U15.23; no longer U14.2, U14.23
- net 3.3V3: now also U20.2, U20.23; no longer U19.2, U19.23
- net 3.3V4: now also U25.2, U25.23; no longer U24.2, U24.23
- net 3.3V5: now also U30.2, U30.23; no longer U29.2, U29.23
- net 3.3V6: now also U35.2, U35.23; no longer U34.2, U34.23
- net 3.3V7: now also U40.2, U40.23; no longer U39.2, U39.23
- net 5V: now also S4.1, S4.4; no longer S3.3
- net 5V1: now also S3.1, S3.4, U9.5V; no longer S6.3, U10.5V
- net 5V2: now also S8.1, S8.4, U14.5V; no longer S9.3, U15.5V
- net 5V3: now also S11.1, S11.4, U19.5V; no longer S12.3, U20.5V
- net 5V4: now also S14.1, S14.4, U24.5V; no longer S15.3, U25.5V
- net 5V5: now also S17.1, S17.4, U29.5V; no longer S18.3, U30.5V
- net 5V6: now also S20.1, S20.4, U34.5V; no longer S21.3, U35.5V
- net 5V7: now also S23.1, S23.4, U39.5V; no longer S24.3, U40.5V
- net CS-IN1: now also U10.14; no longer U9.14
- net CS-IN2: now also U15.14; no longer U14.14
- net CS-IN3: now also U20.14; no longer U19.14
- net CS-IN4: now also U25.14; no longer U24.14
- net CS-IN5: now also U30.14; no longer U29.14
- net CS-IN6: now also U35.14; no longer U34.14
- net CS-IN7: now also U40.14; no longer U39.14
- net CS1: now also U9.D10; no longer U10.D10
- net CS2: now also U14.D10; no longer U15.D10
- net CS3: now also U19.D10; no longer U20.D10
- net CS4: now also U24.D10; no longer U25.D10
- net CS5: now also U29.D10; no longer U30.D10
- net CS6: now also U34.D10; no longer U35.D10
- net CS7: now also U39.D10; no longer U40.D10
- net GND1: now also S1.1, U10.19, U10.3, U9.GND@0, U9.GND@1, U9.GND@2; no longer S4.1, U10.GND@0, U10.GND@1, U10.GND@2, U9.19, U9.3
- net GND2: now also U14.GND@0, U14.GND@1, U14.GND@2, U15.19, U15.3; no longer U14.19, U14.3, U15.GND@0, U15.GND@1, U15.GND@2
- net GND3: now also U19.GND@0, U19.GND@1, U19.GND@2, U20.19, U20.3; no longer U19.19, U19.3, U20.GND@0, U20.GND@1, U20.GND@2
- net GND4: now also U24.GND@0, U24.GND@1, U24.GND@2, U25.19, U25.3; no longer U24.19, U24.3, U25.GND@0, U25.GND@1, U25.GND@2
- net GND5: now also U29.GND@0, U29.GND@1, U29.GND@2, U30.19, U30.3; no longer U29.19, U29.3, U30.GND@0, U30.GND@1, U30.GND@2
- net GND6: now also U34.GND@0, U34.GND@1, U34.GND@2, U35.19, U35.3; no longer U34.19, U34.3, U35.GND@0, U35.GND@1, U35.GND@2
- net GND7: now also U39.GND@0, U39.GND@1, U39.GND@2, U40.19, U40.3; no longer U39.19, U39.3, U40.GND@0, U40.GND@1, U40.GND@2
- net GPIN10: now also U10.31; no longer U9.31
- net GPIN11: now also U10.30; no longer U9.30
- net GPIN12: now also U10.29; no longer U9.29
- net GPIN13: now also U10.28; no longer U9.28
- net GPIN14: now also U10.27; no longer U9.27
- net GPIN15: now also U10.26; no longer U9.26
- net GPIN16: now also U15.1; no longer U14.1
- net GPIN17: now also U15.32; no longer U14.32
- net GPIN18: now also U15.31; no longer U14.31
- net GPIN19: now also U15.30; no longer U14.30
- net GPIN20: now also U15.29; no longer U14.29
- net GPIN21: now also U15.28; no longer U14.28
- net GPIN22: now also U15.27; no longer U14.27
- net GPIN23: now also U15.26; no longer U14.26
- net GPIN24: now also U20.1; no longer U19.1
- net GPIN25: now also U20.32; no longer U19.32
- net GPIN26: now also U20.31; no longer U19.31
- net GPIN27: now also U20.30; no longer U19.30
- net GPIN28: now also U20.29; no longer U19.29
- net GPIN29: now also U20.28; no longer U19.28
- net GPIN30: now also U20.27; no longer U19.27
- net GPIN31: now also U20.26; no longer U19.26
- net GPIN32: now also U25.1; no longer U24.1
- net GPIN33: now also U25.32; no longer U24.32
- net GPIN34: now also U25.31; no longer U24.31
- net GPIN35: now also U25.30; no longer U24.30
- net GPIN36: now also U25.29; no longer U24.29
- net GPIN37: now also U25.28; no longer U24.28
- net GPIN38: now also U25.27; no longer U24.27
- net GPIN39: now also U25.26; no longer U24.26
- net GPIN40: now also U30.1; no longer U29.1
- net GPIN41: now also U30.32; no longer U29.32
- net GPIN42: now also U30.31; no longer U29.31
- net GPIN43: now also U30.30; no longer U29.30
- net GPIN44: now also U30.29; no longer U29.29
- net GPIN45: now also U30.28; no longer U29.28
- net GPIN46: now also U30.27; no longer U29.27
- net GPIN47: now also U30.26; no longer U29.26
- net GPIN48: now also U35.1; no longer U34.1
- net GPIN49: now also U35.32; no longer U34.32
- net GPIN50: now also U35.31; no longer U34.31
- net GPIN51: now also U35.30; no longer U34.30
- net GPIN52: now also U35.29; no longer U34.29
- net GPIN53: now also U35.28; no longer U34.28
- net GPIN54: now also U35.27; no longer U34.27
- net GPIN55: now also U35.26; no longer U34.26
- net GPIN56: now also U40.1; no longer U39.1
- net GPIN57: now also U40.32; no longer U39.32
- net GPIN58: now also U40.31; no longer U39.31
- net GPIN59: now also U40.30; no longer U39.30
- net GPIN60: now also U40.29; no longer U39.29
- net GPIN61: now also U40.28; no longer U39.28
- net GPIN62: now also U40.27; no longer U39.27
- net GPIN63: now also U40.26; no longer U39.26
- net GPIN8: now also U10.1; no longer U9.1
- net GPIN9: now also U10.32; no longer U9.32
- net GPOUT10: now also U10.6; no longer U9.6
- net GPOUT11: now also U10.7; no longer U9.7
- net GPOUT12: now also U10.8; no longer U9.8
- net GPOUT13: now also U10.9; no longer U9.9
- net GPOUT14: now also U10.10; no longer U9.10
- net GPOUT15: now also U10.11; no longer U9.11
- net GPOUT16: now also U15.4; no longer U14.4
- net GPOUT17: now also U15.5; no longer U14.5
- net GPOUT18: now also U15.6; no longer U14.6
- net GPOUT19: now also U15.7; no longer U14.7
- net GPOUT20: now also U15.8; no longer U14.8
- net GPOUT21: now also U15.9; no longer U14.9
- net GPOUT22: now also U15.10; no longer U14.10
- net GPOUT23: now also U15.11; no longer U14.11
- net GPOUT24: now also U20.4; no longer U19.4
- net GPOUT25: now also U20.5; no longer U19.5
- net GPOUT26: now also U20.6; no longer U19.6
- net GPOUT27: now also U20.7; no longer U19.7
- net GPOUT28: now also U20.8; no longer U19.8
- net GPOUT29: now also U20.9; no longer U19.9
- net GPOUT30: now also U20.10; no longer U19.10
- net GPOUT31: now also U20.11; no longer U19.11
- net GPOUT32: now also U25.4; no longer U24.4
- net GPOUT33: now also U25.5; no longer U24.5
- net GPOUT34: now also U25.6; no longer U24.6
- net GPOUT35: now also U25.7; no longer U24.7
- net GPOUT36: now also U25.8; no longer U24.8
- net GPOUT37: now also U25.9; no longer U24.9
- net GPOUT38: now also U25.10; no longer U24.10
- net GPOUT39: now also U25.11; no longer U24.11
- net GPOUT40: now also U30.4; no longer U29.4
- net GPOUT41: now also U30.5; no longer U29.5
- net GPOUT42: now also U30.6; no longer U29.6
- net GPOUT43: now also U30.7; no longer U29.7
- net GPOUT44: now also U30.8; no longer U29.8
- net GPOUT45: now also U30.9; no longer U29.9
- net GPOUT46: now also U30.10; no longer U29.10
- net GPOUT47: now also U30.11; no longer U29.11
- net GPOUT48: now also U35.4; no longer U34.4
- net GPOUT49: now also U35.5; no longer U34.5
- net GPOUT50: now also U35.6; no longer U34.6
- net GPOUT51: now also U35.7; no longer U34.7
- net GPOUT52: now also U35.8; no longer U34.8
- net GPOUT53: now also U35.9; no longer U34.9
- net GPOUT54: now also U35.10; no longer U34.10
- net GPOUT55: now also U35.11; no longer U34.11
- net GPOUT56: now also U40.4; no longer U39.4
- net GPOUT57: now also U40.5; no longer U39.5
- net GPOUT58: now also U40.6; no longer U39.6
- net GPOUT59: now also U40.7; no longer U39.7
- net GPOUT60: now also U40.8; no longer U39.8
- net GPOUT61: now also U40.9; no longer U39.9
- net GPOUT62: now also U40.10; no longer U39.10
- net GPOUT63: now also U40.11; no longer U39.11
- net GPOUT8: now also U10.4; no longer U9.4
- net GPOUT9: now also U10.5; no longer U9.5
- net GPX1: now also U10.17, U9.D8; no longer U10.D8, U9.17
- net GPX2: now also U14.D8, U15.17; no longer U14.17, U15.D8
- net GPX3: now also U19.D8, U20.17; no longer U19.17, U20.D8
- net GPX4: now also U24.D8, U25.17; no longer U24.17, U25.D8
- net GPX5: now also U29.D8, U30.17; no longer U29.17, U30.D8
- net GPX6: now also U34.D8, U35.17; no longer U34.17, U35.D8
- net GPX7: now also U39.D8, U40.17; no longer U39.17, U40.D8
- net INT1: now also U10.18, U9.D9; no longer U10.D9, U9.18
- net INT2: now also U14.D9, U15.18; no longer U14.18, U15.D9
- net INT3: now also U19.D9, U20.18; no longer U19.18, U20.D9
- net INT4: now also U24.D9, U25.18; no longer U24.18, U25.D9
- net INT5: now also U29.D9, U30.18; no longer U29.18, U30.D9
- net INT6: now also U34.D9, U35.18; no longer U34.18, U35.D9
- net INT7: now also U39.D9, U40.18; no longer U39.18, U40.D9
- net MAX_D_N1: now also U10.20; no longer U9.20
- net MAX_D_N2: now also U15.20; no longer U14.20
- net MAX_D_N3: now also U20.20; no longer U19.20
- net MAX_D_N4: now also U25.20; no longer U24.20
- net MAX_D_N5: now also U30.20; no longer U29.20
- net MAX_D_N6: now also U35.20; no longer U34.20
- net MAX_D_N7: now also U40.20; no longer U39.20
- net MAX_D_P1: now also U10.21; no longer U9.21
- net MAX_D_P2: now also U15.21; no longer U14.21
- net MAX_D_P3: now also U20.21; no longer U19.21
- net MAX_D_P4: now also U25.21; no longer U24.21
- net MAX_D_P5: now also U30.21; no longer U29.21
- net MAX_D_P6: now also U35.21; no longer U34.21
- net MAX_D_P7: now also U40.21; no longer U39.21
- net N$2: now also S4.2, S4.5, S5.2, S5.5; no longer S1.2, S3.2
- net N$202: now also S1.3, U9.RES; no longer C14.+, C19.1, R16.2, S6.1, U4.2, U4.4
- net N$306: now also C25.+, C30.1, R26.2, S8.3, S8.6, U11.2, U11.4; no longer S8.2, S9.2
- net N$408: now also S10.3, U19.RES; no longer S11.2, S12.2
- net N$6: now also S4.3, S4.6; no longer S3.1
- net PICO-IN1: now also U10.16; no longer U9.16
- net PICO-IN2: now also U15.16; no longer U14.16
- net PICO-IN3: now also U20.16; no longer U19.16
- net PICO-IN4: now also U25.16; no longer U24.16
- net PICO-IN5: now also U30.16; no longer U29.16
- net PICO-IN6: now also U35.16; no longer U34.16
- net PICO-IN7: now also U40.16; no longer U39.16
- net PICO1: now also U9.D11; no longer U10.D11
- net PICO2: now also U14.D11; no longer U15.D11
- net PICO3: now also U19.D11; no longer U20.D11
- net PICO4: now also U24.D11; no longer U25.D11
- net PICO5: now also U29.D11; no longer U30.D11
- net PICO6: now also U34.D11; no longer U35.D11
- net PICO7: now also U39.D11; no longer U40.D11
- net POCI1: now also U10.15, U9.D12; no longer U10.D12, U9.15
- net POCI2: now also U14.D12, U15.15; no longer U14.15, U15.D12
- net POCI3: now also U19.D12, U20.15; no longer U19.15, U20.D12
- net POCI4: now also U24.D12, U25.15; no longer U24.15, U25.D12
- net POCI5: now also U29.D12, U30.15; no longer U29.15, U30.D12
- net POCI6: now also U34.D12, U35.15; no longer U34.15, U35.D12
- net POCI7: now also U39.D12, U40.15; no longer U39.15, U40.D12
- net RESET-IN1: now also U10.12; no longer U9.12
- net RESET-IN2: now also U15.12; no longer U14.12
- net RESET-IN3: now also U20.12; no longer U19.12
- net RESET-IN4: now also U25.12; no longer U24.12
- net RESET-IN5: now also U30.12; no longer U29.12
- net RESET-IN6: now also U35.12; no longer U34.12
- net RESET-IN7: now also U40.12; no longer U39.12
- net RESET1: now also U9.D7; no longer U10.D7
- net RESET2: now also U14.D7; no longer U15.D7
- net RESET3: now also U19.D7; no longer U20.D7
- net RESET4: now also U24.D7; no longer U25.D7
- net RESET5: now also U29.D7; no longer U30.D7
- net RESET6: now also U34.D7; no longer U35.D7
- net RESET7: now also U39.D7; no longer U40.D7
- net SCK-IN1: now also U10.13; no longer U9.13
- net SCK-IN2: now also U15.13; no longer U14.13
- net SCK-IN3: now also U20.13; no longer U19.13
- net SCK-IN4: now also U25.13; no longer U24.13
- net SCK-IN5: now also U30.13; no longer U29.13
- net SCK-IN6: now also U35.13; no longer U34.13
- net SCK-IN7: now also U40.13; no longer U39.13
- net SCK1: now also U9.D13; no longer U10.D13
- net SCK2: now also U14.D13; no longer U15.D13
- net SCK3: now also U19.D13; no longer U20.D13
- net SCK4: now also U24.D13; no longer U25.D13
- net SCK5: now also U29.D13; no longer U30.D13
- net SCK6: now also U34.D13; no longer U35.D13
- net SCK7: now also U39.D13; no longer U40.D13
- net VBCOMP1: now also U10.22; no longer U9.22
- net VBCOMP2: now also U15.22; no longer U14.22
- net VBCOMP3: now also U20.22; no longer U19.22
- net VBCOMP4: now also U25.22; no longer U24.22
- net VBCOMP5: now also U30.22; no longer U29.22
- net VBCOMP6: now also U35.22; no longer U34.22
- net VBCOMP7: now also U40.22; no longer U39.22
- net VDD: now also S5.3, S5.6; no longer S1.1
- net VDD1: now also S6.3, S6.6; no longer S5.1
- net VDD2: now also S9.3, S9.6; no longer S8.1
- net VDD3: now also S12.3, S12.6; no longer S11.1
- net VDD4: now also S15.3, S15.6; no longer S14.1
- net VDD5: now also S18.3, S18.6; no longer S17.1
- net VDD6: now also S21.3, S21.6; no longer S20.1
- net VDD7: now also S24.3, S24.6; no longer S23.1
- net VIN1: now also U9.VIN; no longer U10.VIN
- net VIN2: now also U14.VIN; no longer U15.VIN
- net VIN3: now also U19.VIN; no longer U20.VIN
- net VIN4: now also U24.VIN; no longer U25.VIN
- net VIN5: now also U29.VIN; no longer U30.VIN
- net VIN6: now also U34.VIN; no longer U35.VIN
- net VIN7: now also U39.VIN; no longer U40.VIN
- net XI1: now also U10.24; no longer U9.24
- net XI2: now also U15.24; no longer U14.24
- net XI3: now also U20.24; no longer U19.24
- net XI4: now also U25.24; no longer U24.24
- net XI5: now also U30.24; no longer U29.24
- net XI6: now also U35.24; no longer U34.24
- net XI7: now also U40.24; no longer U39.24
- net XO1: now also U10.25; no longer U9.25
- net XO2: now also U15.25; no longer U14.25
- net XO3: now also U20.25; no longer U19.25
- net XO4: now also U25.25; no longer U24.25
- net XO5: now also U30.25; no longer U29.25
- net XO6: now also U35.25; no longer U34.25
- net XO7: now also U40.25; no longer U39.25
Routing:
- net N$814: track 30.6 -> 0.00 mm, vias 0 -> 1
- net N$712: track 30.6 -> 0.00 mm, vias 0 -> 1
- net N$610: track 30.6 -> 0.00 mm, vias 0 -> 1
- net N$406: track 30.6 -> 0.00 mm, vias 0 -> 1
- net N$508: track 30.6 -> 0.00 mm, vias 0 -> 1
- net N$304: track 30.6 -> 0.00 mm, vias 0 -> 1
- net N$6: track 30.6 -> 4.75 mm, vias 0 -> 18
- net N$202: track 30.6 -> 7.09 mm
- net N$617: track 0.00 -> 13.4 mm, vias 1 -> 0
- net N$514: track 0.00 -> 13.4 mm, vias 1 -> 0
- net N$411: track 0.00 -> 13.4 mm, vias 1 -> 0
- net N$308: track 0.00 -> 13.4 mm
- net N$205: track 0.00 -> 13.4 mm
- net N$823: track 0.00 -> 13.4 mm
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- added copper zone on layer 1, net N$203
- added copper zone on layer 16, net N$203
- added copper zone on layer 1, net N$306
- added copper zone on layer 16, net N$306
- added copper zone on layer 1, net N$409
- added copper zone on layer 16, net N$409
- added copper zone on layer 1, net N$512
- added copper zone on layer 16, net N$512
- added copper zone on layer 1, net N$6
- added copper zone on layer 16, net N$6
- added copper zone on layer 1, net N$615
- added copper zone on layer 16, net N$615
- added copper zone on layer 1, net N$718
- added copper zone on layer 16, net N$718
- added copper zone on layer 1, net N$821
- added copper zone on layer 16, net N$821

Commit message: Changed R4 and R5 resistors
Changed the value of R4 and R5 from 2.2k to 10k for fixing the LED power off issue from testing. Changed the schematic, board, and panel files for consistency across the project.
Parts:
- R17, R18, R27, R28, R37, R38, R47, R48, R57, R58, R67, R68, R77, R78: value 2.2k -> 56k
- R19, R20, R29, R30, R39, R40, R49, R50, R59, R60, R69, R70, R79, R80: value 56k -> 10k
- R4, R5: value 2.2k -> 10k
- moved R17 35.5 mm to (93.2, 50.8), turned to 270 degrees
- moved R19 35.5 mm to (63.2, 31.8), turned to 180 degrees
- moved R37 35.5 mm to (93.2, 118.9), turned to 270 degrees
- moved R39 35.5 mm to (63.2, 99.8), turned to 180 degrees
- moved R27 35.5 mm to (39.4, 118.9), turned to 270 degrees
- moved R29 35.5 mm to (9.40, 99.8), turned to 180 degrees
- moved R57 35.5 mm to (93.2, 186.9), turned to 270 degrees
- moved R59 35.5 mm to (63.2, 167.9), turned to 180 degrees
- moved R77 35.5 mm to (93.2, 255.0), turned to 270 degrees
- moved R79 35.5 mm to (63.2, 236.0), turned to 180 degrees
- moved R47 35.5 mm to (39.4, 186.9), turned to 270 degrees
- moved R49 35.5 mm to (9.40, 167.9), turned to 180 degrees
- moved R67 35.5 mm to (39.4, 255.0), turned to 270 degrees
- moved R69 35.5 mm to (9.40, 236.0), turned to 180 degrees
- moved R68 34.9 mm to (33.7, 254.9), turned to 270 degrees
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Connections:
- net 3.3V1: now also R19.2, R20.2; no longer R17.2, R18.2
- net 3.3V2: now also R29.2, R30.2; no longer R27.2, R28.2
- net 3.3V3: now also R39.2, R40.2; no longer R37.2, R38.2
- net 3.3V4: now also R49.2, R50.2; no longer R47.2, R48.2
- net 3.3V5: now also R59.2, R60.2; no longer R57.2, R58.2
- net 3.3V6: now also R69.2, R70.2; no longer R67.2, R68.2
- net 3.3V7: now also R79.2, R80.2; no longer R77.2, R78.2
- net CC10: now also R48.1; no longer R50.1
- net CC11: now also R57.1; no longer R59.1
- net CC12: now also R58.1; no longer R60.1
- net CC13: now also R67.1; no longer R69.1
- net CC14: now also R68.1; no longer R70.1
- net CC15: now also R77.1; no longer R79.1
- net CC16: now also R78.1; no longer R80.1
- net CC3: now also R17.1; no longer R19.1
- net CC4: now also R18.1; no longer R20.1
- net CC5: now also R27.1; no longer R29.1
- net CC6: now also R28.1; no longer R30.1
- net CC7: now also R37.1; no longer R39.1
- net CC8: now also R38.1; no longer R40.1
- net CC9: now also R47.1; no longer R49.1
- net CS1: now also R20.1; no longer R18.1
- net CS2: now also R30.1; no longer R28.1
- net CS3: now also R40.1; no longer R38.1
- net CS4: now also R50.1; no longer R48.1
- net CS5: now also R60.1; no longer R58.1
- net CS6: now also R70.1; no longer R68.1
- net CS7: now also R80.1; no longer R78.1
- net RESET1: now also R19.1; no longer R17.1
- net RESET2: now also R29.1; no longer R27.1
- net RESET3: now also R39.1; no longer R37.1
- net RESET4: now also R49.1; no longer R47.1
- net RESET5: now also R59.1; no longer R57.1
- net RESET6: now also R69.1; no longer R67.1
- net RESET7: now also R79.1; no longer R77.1
- net VDD1: now also R17.2, R18.2; no longer R19.2, R20.2
- net VDD2: now also R27.2, R28.2; no longer R29.2, R30.2
- net VDD3: now also R37.2, R38.2; no longer R39.2, R40.2
- net VDD4: now also R47.2, R48.2; no longer R49.2, R50.2
- net VDD5: now also R57.2, R58.2; no longer R59.2, R60.2
- net VDD6: now also R67.2, R68.2; no longer R69.2, R70.2
- net VDD7: now also R77.2, R78.2; no longer R79.2, R80.2
